Commit message: Working solution

File: 3DoFRobot.urdf (robot description, URDF)
Before this commit: robot robot, 5 links, 4 joints
Joints:
- joint Joint_1: limit lower=-12.96705972839 upper=12.96705972839 effort=204 velocity=100.91986217719 -> lower=-100 upper=100 effort=204 velocity=100.91986217719
- joint Joint_2: limit lower=-2.96705972839 upper=2.96705972839 effort=204 velocity=1.91986217719 -> lower=-100 upper=100 effort=204 velocity=100
- joint Joint_3: limit lower=-2.96705972839 upper=2.96705972839 effort=204 velocity=1.91986217719 -> lower=-100 upper=100 effort=204 velocity=100
